File: hardware/esp32-alarmlicht.kicad_sch (KiCad schematic)
At the start: 14 parts, among them J102 LGRA, SW101 Funklicht

Commit message: wip: readme; schematics done
Parts:
- EXT1: symbol ESP32-EVB_Rev_K1:BH40S -> Connector_Generic:Conn_02x20_Odd_Even
- PWR2: symbol ESP32-EVB_Rev_K1:CON2 -> Connector_Generic:Conn_01x02
Connections:
- no-connect marks 28 -> 29
Other:
- title: (none) -> ESP32-Alarmlicht
